Commit message: camera working in moderate form b

File: models/turtlebot3_burger.urdf (robot description, URDF)
Before this commit: robot turtlebot3_burger, 5 links, 4 joints
Links:
- added link camera_link
- added link camera_link_optical
- added link laser
Joints:
- added joint camera_joint: type fixed, parent base_link, child camera_link, origin xyz=0.09 0 0.08
- added joint camera_optical_joint: type fixed, parent camera_link, child camera_link_optical, origin rpy=-1.5708 0 -1.5708
- added joint laser_joint: type fixed, parent base_link, child laser, origin xyz=0 0 0.04
